File: teensy-toslink-receiver.kicad_pcb (KiCad board)
At the start: 2 copper layers, 24.9 x 18.3 mm, 11 parts, among them J1 Conn_01x03, J2 Conn_01x05, J3 Conn_01x05, J4 Conn_01x05, J5 Conn_01x03, J6 Conn_01x04, J7 HDMI_A_1.4, U1 PLR135-T10

Commit message: gerbers: Add gerbers
* Sent to OSHPark with zip timestamp 1605504464
* $3.50 for 3x shipped.
Other:
- board text added: "wut a mess"
Changed lines of the file:
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@@
   (general
     (thickness 1.6)
-    (drawings 8)
-    (tracks 60)
+    (drawings 9)
+    (tracks 59)
     (zones 0)
     (modules 11)
@@
     (visible_elements FFFDFF7F)
     (pcbplotparams
-      (layerselection 0x010fc_ffffffff)
+      (layerselection 0x010f0_ffffffff)
       (usegerberextensions false)
       (usegerberattributes true)
@@
       (plotinvisibletext false)
       (padsonsilk false)
-      (subtractmaskfromsilk false)
+      (subtractmaskfromsilk true)
       (outputformat 1)
       (mirror false)
-      (drillshape 1)
+      (drillshape 0)
       (scaleselection 1)
-      (outputdirectory ""))
+      (outputdirectory "gerbers"))
   )
   (net 0 "")
@@
     )
   )
+  (gr_text "wut a mess" (at 137.287 73.66 90) (layer B.SilkS)
+    (effects (font (size 1.5 1.5) (thickness 0.3)) (justify mirror))
+  )
   (gr_line (start 159.004 81.534) (end 159.004 65.786) (layer Edge.Cuts) (width 0.05))
   (gr_arc (start 157.734 65.786) (end 157.734 64.516) (angle 90) (layer Edge.Cuts) (width 0.05))
@@
   (segment (start 149.24 74.799625) (end 149.6525 74.387125) (width 0.25) (layer B.Cu) (net 2))
   (segment (start 149.24 76.2) (end 149.24 74.799625) (width 0.25) (layer B.Cu) (net 2))
-  (segment (start 141.323 71.91) (end 139.982 71.91) (width 0.25) (layer F.Cu) (net 3))
-  (segment (start 139.982 71.91) (end 139.7 71.628) (width 0.25) (layer F.Cu) (net 3))
-  (segment (start 139.7 71.628) (end 139.7 69.088) (width 0.25) (layer F.Cu) (net 3))
-  (segment (start 139.7 69.088) (end 140.208 68.58) (width 0.25) (layer F.Cu) (net 3))
-  (segment (start 140.208 68.58) (end 142.24 68.58) (width 0.25) (layer F.Cu) (net 3))
-  (segment (start 144.78 66.04) (end 147.32 66.04) (width 0.25) (layer F.Cu) (net 3))
-  (segment (start 142.24 68.58) (end 144.78 66.04) (width 0.25) (layer F.Cu) (net 3))
   (segment (start 141.323 71.91) (end 140.18 71.91) (width 0.25) (layer F.Cu) (net 3))
-  (segment (start 140.18 71.91) (end 139.7 72.39) (width 0.25) (layer F.Cu) (net 3))
-  (segment (start 139.7 72.39) (end 139.7 78.994) (width 0.25) (layer F.Cu) (net 3))
-  (segment (start 139.7 78.994) (end 140.208 79.502) (width 0.25) (layer F.Cu) (net 3))
-  (segment (start 140.208 79.502) (end 143.002 79.502) (width 0.25) (layer F.Cu) (net 3))
-  (segment (start 143.002 79.502) (end 143.51 80.01) (width 0.25) (layer F.Cu) (net 3))
   (segment (start 146.05 80.01) (end 147.32 81.28) (width 0.25) (layer F.Cu) (net 3))
   (segment (start 143.51 80.01) (end 146.05 80.01) (width 0.25) (layer F.Cu) (net 3))
+  (segment (start 143.002 79.502) (end 143.51 80.01) (width 0.25) (layer F.Cu) (net 3))
+  (segment (start 140.208 79.502) (end 143.002 79.502) (width 0.25) (layer F.Cu) (net 3))
+  (segment (start 139.7 78.994) (end 140.208 79.502) (width 0.25) (layer F.Cu) (net 3))
+  (segment (start 140.208 68.58) (end 139.7 69.088) (width 0.25) (layer F.Cu) (net 3))
+  (segment (start 142.24 68.58) (end 140.208 68.58) (width 0.25) (layer F.Cu) (net 3))
+  (segment (start 144.78 66.04) (end 142.24 68.58) (width 0.25) (layer F.Cu) (net 3))
+  (segment (start 147.32 66.04) (end 144.78 66.04) (width 0.25) (layer F.Cu) (net 3))
+  (segment (start 139.728 71.91) (end 139.7 71.882) (width 0.25) (layer F.Cu) (net 3))
+  (segment (start 141.323 71.91) (end 139.728 71.91) (width 0.25) (layer F.Cu) (net 3))
+  (segment (start 139.7 71.882) (end 139.7 78.994) (width 0.25) (layer F.Cu) (net 3))
+  (segment (start 139.7 69.088) (end 139.7 71.882) (width 0.25) (layer F.Cu) (net 3))
   (segment (start 149.86 66.04) (end 149.86 68.58) (width 0.25) (layer F.Cu) (net 4))
   (segment (start 152.4 66.04) (end 152.4 66.548) (width 0.25) (layer F.Cu) (net 5))
